File: Projekt tutorial.sch (KiCad schematic (older format))
At the start: 50 parts, among them P1 Silnik1, P2 CONN_01X02, P3 Silnik2, P4 Programator, SW1 SWITCH, U1 LM1117, U10 STM32F030K6, U11 KTIR0711S, U2 TB6612, U3 TB6612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

Commit message: Sharpy analogowe, microUSB
Parts:
- removed C10, C7, C8, C9: C, symbol C
- removed D1, D2, D3, D4: LED, symbol LED
- removed P4: Programator, symbol CONN_01X04
- removed R1, R2, R3, R4: R, symbol R
- removed U5, U6, U7, U8: SHARP_40CM, Battery_Holders:Keystone_2468_2xAAA, symbol SHARP_40CM
- added P?: USB_OTG, symbol USB_OTG
- added P? (x4): Sharp analog., symbol CONN_01X03
- P2: value CONN_01X02 -> zlacze z kluczem
- R5, R7: value R -> 200
- R6, R8: value R -> 20k
- SW1: value SWITCH -> wlacznik
Connections:
- net +3V3: now also P?.1 (VCC)
- net +5V: now also P?.1 (P1), P?.1 (P1), P?.1 (P1), P?.1 (P1)
- net GND: now also P?.3 (P3), P?.3 (P3), P?.3 (P3), P?.3 (P3), P?.5 (GND), P?.6 (shield)
- net PROG1: no longer names the net of U10.26 (SPI1_SCK/EVENTOUT/PB3)
- net PROG2: no longer names the net of U10.27 (SPI1_MISO/TIM3_CH1/EVENTOUT/PB4)
- net PROG3: no longer names the net of U10.28 (SPI1_MOSI/I2C1_SMBA/TIM16_BKIN/TIM3_CH2/PB5)
- net PROG4 renamed RESET
- net RESET: now also P?.3 (D+)
- net SHARP1 renamed V01
- net V01: now also P?.2 (P2)
- net SHARP2 renamed V02
- net V02: now also P?.2 (P2)
- net SHARP3 renamed V03
- net V03: now also P?.2 (P2)
- net SHARP4 renamed V04
- net V04: now also P?.2 (P2)
- new net CLC: P?.4 (ID)
- new net TMS: P?.2 (D-)
