File: Projekt tutorial.sch (KiCad schematic (older format))
At the start: 29 parts, among them P1 CONN_01X02, SW1 SWITCH, U1 LM1117, U2 LM1117, U3 KTIR0711S, U4 SHARP_40CM

Commit message: Podłączenie mostków, dodanie programatora do schematu
Parts:
- removed C?: CP, symbol CP
- removed C?: C, symbol C
- removed U? (x2): L293D, symbol L293D
- added 100n (x2), 100n? (x2), 10u, 10u?, C? (x3): C, symbol C
- added C? (x2): 22uF, symbol CP1
- added D? (x3): LED, symbol LED
- added P?: Silnik 1, symbol CONN_01X03
- added P?: Silnik 2, symbol CONN_01X03
- added P?: Programator, symbol CONN_01X04
- added R? (x3): R, symbol R
- added U? (x2): TB6612, symbol TB6612
- added U? (x3): SHARP_40CM, Battery_Holders:Keystone_2468_2xAAA, symbol SHARP_40CM
Connections:
- net labels added: IN1, IN2, IN3, IN4, M_OUT1, M_OUT2, M_OUT3, M_OUT4, PROG1, PROG2, PROG3, PROG4, PWM, SHARP1, SHARP2, SHARP3, SHARP4, VDD
- net labels removed: +BATT
- wire segments 77 -> 162
Other:
- moved on the sheet: C1, C2, C3, C4, C?, D?, P1, R2, R3, R?, SW1, U1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

Commit message: Wprowadzone poprawki od Szymona
Parts:
- removed P?: Silnik 1, symbol CONN_01X03
- removed P?: Silnik 2, symbol CONN_01X03
- added P1: Silnik1, symbol CONN_01X02
- added P3: Silnik2, symbol CONN_01X02
- C16: renamed from 10u?; value C -> 10uF
- C17: renamed from 10u; value C -> 10uF
- C18, C20: renamed from 100n?; value C -> 100nF
- C19, C21: renamed from 100n; value C -> 100nF
- gave numbers to parts that had none: 26
- renumbered C2 to C1, C5 to C11, C6 to C12, C7 to C13, C8 to C14, C1 to C2, C4 to C3, C3 to C4, P1 to P2, R2 to R5, R3 to R6, U2 to U1, U1 to U4, U4 to U5, U3 to U9
Connections:
- net +3V3: now also U2.19 (STBY), U2.20 (VCC)
- net +7,4V: no longer P2.2 (P2)
- net GND: now also P2.2 (P2)
- net M_OUT1: now also P1.1 (P1); no longer U2.5 (AO2), U2.6 (AO2), U2.7 (BO2), U2.8 (BO2)
- net M_OUT3: now also P3.1 (P1); no longer U3.5 (AO2), U3.6 (AO2), U3.7 (BO2), U3.8 (BO2)
- net VDD: no longer U2.19 (STBY), U2.20 (VCC)
- new net M_OUT2: P1.2 (P2), U2.5 (AO2), U2.6 (AO2), U2.7 (BO2), U2.8 (BO2)
- new net M_OUT4: P3.2 (P2), U3.5 (AO2), U3.6 (AO2), U3.7 (BO2), U3.8 (BO2)

Commit message: Add files via upload
Dodałem wartości rezystorów, dławika i kondensatorów. Wziąłem je z datasheetów, ale nie wiem czy są poprawne w naszym konkretnym przypadku :P Poprawiłem ogólnie trochę rzeczy na schemacie, ale gdy chce go zdebugować wyrzuca ciągle błędy, że pin nie jest sterowany czy coś w tym stylu :/
Parts:
- removed P2: CONN_01X02, Socket_Strips:Socket_Strip_Straight_1x02, symbol CONN_01X02
- removed SW1: SWITCH, symbol SWITCH
- removed U1, U4: LM1117, symbol LM1117
- added BT1: Bateria 7,4 V, symbol Battery
- added P1: Wtyczka do zasilania, symbol CONN_02X02
- added U1: LM1117-5.0, symbol LM1117-5.0
- added U4: LM1117-3.3, symbol LM1117-3.3
- C1: value CP -> 10uF
- C10, C7, C8, C9: value C -> 0,1uF
- C11: value CP -> 100nF
- C12, C13, C14, C15: value C -> 100nF
- C2: value 100uF -> 10uF
- C3: value CP -> 100uF
- L1: value L_Small -> 10uH
- R1, R2, R3, R4: value R -> 1 Ω
- R5, R7: value R -> 200Ω
- R6, R8: value R -> 20kΩ
- renumbered P1 to S1, P3 to S2
Connections:
- net +3V3: now also C16.2, C18.2, U4.2 (VO), U4.4 (VO); no longer L1.1, U10.1 (VDD)
- net +5V: now also U1.2 (VO), U1.4 (VO), U4.3 (VI)
- net +7,4V: now also P1.2 (P2), U1.3 (VI)
- net GND: now also C10.2, C9.2, P1.4 (P4), U1.1 (GND/ADJ), U4.1 (GND/ADJ); no longer C10.1, C9.1
- net SHARP1: now also U5.3 (VO)
- net SHARP2: now also U6.3 (VO)
- net SHARP3: now also U7.3 (VO)
- net SHARP4: now also U8.3 (VO)
- net VDD: now also C17.2, C19.2
- net at U7.5 (REG): now also C9.1; no longer C9.2
- net at U8.5 (REG): now also C10.1; no longer C10.2
- removed net sharp: U5.3 (VO), U6.3 (VO), U7.3 (VO), U8.3 (VO)
- new net: L1.1, U10.1 (VDD)
- new net: BT1.1, P1.1 (P1)
- new net: BT1.2, P1.3 (P3)
- no-connect marks 1 -> 13
